Commit message: creation of package to spawn my rb1 robot in gazebo

File: my_rb1_description/urdf/my_rb1_robot.urdf (robot description, URDF)
Before this commit: robot rb1_robot, 7 links, 6 joints
Links:
- link back_caster: mass None -> 0.5
- link base_link: mass None -> 22
- link front_caster: mass None -> 0.5
- link left_wheel: mass None -> 1
- link right_wheel: mass None -> 1
Joints:
- joint joint_base_link_back_caster: origin xyz=-0.1 0.0 -0.15 rpy=0.0 0.0 0.0 -> xyz=-0.1 0 -0.15 rpy=0 0 0
- joint joint_base_link_base_footprint: origin xyz=0.0 0.0 -0.15 rpy=0.0 0.0 0.0 -> xyz=0 0 -0.15 rpy=0 0 0
- joint joint_base_link_front_caster: origin xyz=0.1 0.0 -0.15 rpy=0.0 0.0 0.0 -> xyz=0.1 0 -0.15 rpy=0 0 0
- joint joint_base_link_front_laser: origin xyz=0.25 0.0 0.075 rpy=3.1415 0.0 0.0 -> xyz=0.25 0 0.075 rpy=3.1415 0 0
- joint joint_base_link_left_wheel: origin xyz=0.0 0.2 -0.15 rpy=0.0 0.0 0.0 -> xyz=0 0.2 -0.15 rpy=0 0 0
- joint joint_base_link_right_wheel: origin xyz=0.0 -0.2 -0.15 rpy=0.0 0.0 0.0 -> xyz=0 -0.2 -0.15 rpy=0 0 0

Commit message: add diff drive + laser scan gazebo plugin

File: my_rb1_description/urdf/my_rb1_robot.urdf (robot description, URDF)
Before this commit: robot rb1_robot, 7 links, 6 joints
Joints:
- removed joint joint_base_link_base_footprint
- added joint joint_base_footprint_base_link: type fixed, parent base_footprint, child base_link, origin xyz=0 0 -0.15 rpy=0 0 0

Commit message: add modification to the description of the robot

File: my_rb1_description/urdf/my_rb1_robot.urdf (robot description, URDF)
Before this commit: robot rb1_robot, 7 links, 6 joints
Links:
- link left_wheel: mass 1 -> 1.0; geometry collision cylinder length=0.02 radius=0.03; visual cylinder length=0.02 radius=0.03
- link right_wheel: geometry collision cylinder length=0.02 radius=0.03; visual cylinder length=0.02 radius=0.03

Commit message: rename the lase_scan topic to scan

File: my_rb1_description/urdf/my_rb1_robot.urdf (robot description, URDF)
Before this commit: robot rb1_robot, 7 links, 6 joints
Links:
- link left_wheel: geometry collision cylinder length=0.02 radius=0.0275; visual cylinder length=0.02 radius=0.0275
- link right_wheel: geometry collision cylinder length=0.02 radius=0.0275; visual cylinder length=0.02 radius=0.0275
